File: uberdashboard.kicad_pcb (KiCad board)
At the start: 2 copper layers, 44 parts, among them CON1 TOUCH-BM10NB(0.8)-10DS-0.4V(5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, CON2 AMOLED-BM10NB(0.8)-40DS-0.4V(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, M1 VID23-03, M2 VID23-03, P1 CONN_ROUNDX07, Q1 BC817-40, U1 EM63A165TS, U2 STM32F429II, U3 MX25L3206E, U4 MCP2551-I/SN, U5 MCP23008, U6 STOD13AS, U7 LD1117S50TR, U8 LD1117S33TR, Y1 32.768, Y2 8MHz

Commit message: Added files via upload
Parts:
- C11, C12, C13, C2, C4, C6, CON2, L2, L3, Q1, R3, R6, R7, R8, U6: moved to B.Cu
- moved U1 130.4 mm to (84.0, 21.0), turned to 270 degrees
- moved C11 129.1 mm to (47.0, 23.0), turned to 270 degrees
- moved C13 116.1 mm to (51.0, 19.0)
- moved R8 109.7 mm to (61.0, 32.0), turned to 270 degrees
- moved R6 108.5 mm to (50.0, 28.0), turned to 90 degrees
- moved U6 106.4 mm to (51.0, 23.0)
- moved Q1 106.2 mm to (53.0, 28.0)
- moved CON2 104.8 mm to (52.0, 33.0)
- moved L2 103.9 mm to (43.0, 26.0), turned to 270 degrees
- moved U2 103.5 mm to (52.0, 30.0)
- moved L3 102.5 mm to (59.0, 24.0), turned to 90 degrees
- moved M2 100.4 mm to (135.0, 30.0), turned to 90 degrees
- moved C12 98.9 mm to (55.0, 22.0), turned to 90 degrees
- moved Y2 98.7 mm to (27.0, 30.0)
- moved R7 97.8 mm to (58.0, 29.0), turned to 180 degrees
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Other:
- board outline added: 150 x 60 mm

Commit message: right export
Parts:
- added BT1: 3V, Connect:GS2, F.Cu at (78.0, 56.0)
- added C18: C, Capacitors_SMD:C_0603, F.Cu at (81.0, 34.0)
- added C19: 2.2uF, Capacitors_SMD:C_0603, F.Cu at (69.0, 26.0)
- added C20: C, Capacitors_SMD:C_0603, F.Cu at (85.0, 56.0)
- added C21: 2.2uF, Capacitors_SMD:C_0603, F.Cu at (25.0, 46.0)
- added C22: C, Capacitors_SMD:C_0603, F.Cu at (57.0, 57.0)
- added C23: C, Capacitors_SMD:C_0603, F.Cu at (77.0, 41.0)
- added C24: 10uF, Capacitors_SMD:c_elec_4x5.3, F.Cu at (72.0, 34.0)
- added C25: C, Capacitors_SMD:C_0603, F.Cu at (69.0, 40.0)
- added C26: C, Capacitors_SMD:C_0603, F.Cu at (76.0, 26.0)
- added C27: C, Capacitors_SMD:C_0603, F.Cu at (122.0, 44.0)
- added C28, C32, C33: C, Capacitors_SMD:C_0603, F.Cu at (75.0, 70.1)
- added C29: 10uF, Capacitors_SMD:c_elec_4x5.3, F.Cu at (66.0, 54.0)
- added C30: 10uF, Capacitors_SMD:c_elec_4x5.3, F.Cu at (95.0, 48.0)
- added C31: 10uF, Capacitors_SMD:c_elec_4x5.3, F.Cu at (33.0, 53.0)
- added P2: CONN_ROUNDX07, Pin_Headers:Pin_Header_Straight_1x07, F.Cu at (43.0, 2.00)
- C1: value 2.2uF -> 10uF
- C10: value 2.2uF -> C
- C11, C14, C15, C16, C17: value 10uF -> C
- C12: value 2x10uF -> C
- C13, C8: value 1uF -> C
- C2, C3: value 6.8pF -> 1uF
- C4: value 20pF -> 100nF
- C6: value 1uF -> 20pF
- C7: value 100nF -> C
- C9: value 100nF -> 2x10uF
- CON1: value TOUCH-BM10NB(0.8)-10DS-0.4V(51) -> AMOLED-BM10NB(0.8)-40DS-0.4V(51)
- CON2: value AMOLED-BM10NB(0.8)-40DS-0.4V(51) -> TOUCH-BM10NB(0.8)-10DS-0.4V(51)
- P1: value CONN_ROUNDX07 -> CONN_01X06
- R1: value 0 -> 10K
- R2: value 0 -> 10k
- R5: value R -> 1K
- U1: value EM63A165TS -> STOD13AS
- U2: value STM32F429II -> STM32F429ZIT6
- U3: value MX25L3206E -> MCP2551-I/SN
- U4: value MCP2551-I/SN -> LD1117S50TR
- U5: value MCP23008 -> PCA9555
- U6: value STOD13AS -> LD1117S33TR
- U7: value LD1117S50TR -> EM63A165TS
- U8: value LD1117S33TR -> MX25L3206E
- Y1: value 32.768 -> 8MHz
- Y2: value 8MHz -> 32 kHz
Connections:
- C1 pad 1: GND -> Net-(C1-Pad1)
- C1 pad 2: Net-(C1-Pad2) -> GND
- C10 pad 1: Net-(C10-Pad1) -> GND
- C10 pad 2: GND -> Net-(BT1-Pad1)
- C11 pad 1: Net-(C11-Pad1) -> GND
- C11 pad 2: GND -> VDD
- C12 pad 1: Net-(C12-Pad1) -> VDD
- C13 pad 1: Net-(C13-Pad1) -> VDD
- C14 pad 1: +12V -> VDD
- C15 pad 1: +5V -> VDD
- C16 pad 1: +12V -> GND
- C16 pad 2: GND -> VDD
- C17 pad 1: VDD -> GND
- C17 pad 2: GND -> VDD
- C4 pad 1: Net-(C4-Pad1) -> Net-(C3-Pad1)
- C6 pad 1: GND -> Net-(C6-Pad1)
- C6 pad 2: Net-(C6-Pad2) -> GND
- C7 pad 1: GND -> Net-(C7-Pad1)
- C7 pad 2: Net-(C6-Pad2) -> GND
- C9 pad 1: Net-(C8-Pad1) -> Net-(C9-Pad1)
- CON1 pad 1: GND -> Net-(C1-Pad1)
- CON1 pad 2: Net-(CON1-Pad2) -> Net-(C9-Pad1)
- CON1 pad 3: +5V -> Net-(C1-Pad1)
- CON1 pad 4: Net-(CON1-Pad4) -> Net-(C9-Pad1)
- CON1 pad 5: +5V -> VDD
- CON1 pad 7: /SCL -> VDD
- CON1 pad 8: /SDA -> /PCLK
- CON1 pad 9: /IRQ -> /HSYNC
- CON2 pad 1: Net-(C11-Pad1) -> GND
- CON2 pad 11: /VSYNC -> (no net)
- CON2 pad 12: /EN -> (no net)
- CON2 pad 13: Net-(CON2-Pad13) -> (no net)
- CON2 pad 14: GND -> (no net)
- CON2 pad 15: /RESETB -> (no net)
- CON2 pad 16: VDD -> (no net)
- CON2 pad 17: /R5 -> (no net)
- CON2 pad 18: /R4 -> (no net)
- CON2 pad 19: /R3 -> (no net)
- CON2 pad 2: Net-(C12-Pad1) -> Net-(CON2-Pad2)
- CON2 pad 20: /R2 -> (no net)
- CON2 pad 21: /R1 -> (no net)
- CON2 pad 22: /R0 -> (no net)
- CON2 pad 23: /G5 -> (no net)
- CON2 pad 24: /G4 -> (no net)
- CON2 pad 25: /G3 -> (no net)
- CON2 pad 26: /G2 -> (no net)
- CON2 pad 27: /G1 -> (no net)
- CON2 pad 28: /G0 -> (no net)
- CON2 pad 29: /B5 -> (no net)
- CON2 pad 3: Net-(C11-Pad1) -> +5V
- CON2 pad 30: /B4 -> (no net)
- CON2 pad 31: /B3 -> (no net)
- CON2 pad 32: /B2 -> (no net)
- CON2 pad 33: /B1 -> (no net)
- CON2 pad 34: /B0 -> (no net)
- CON2 pad 35: /SDI -> (no net)
- CON2 pad 36: Net-(CON2-Pad36) -> (no net)
- CON2 pad 37: /CSB -> (no net)
- CON2 pad 38: GND -> (no net)
- CON2 pad 39: GND -> (no net)
- CON2 pad 4: Net-(C12-Pad1) -> Net-(CON2-Pad4)
- CON2 pad 40: /SCL -> (no net)
- CON2 pad 5: VDD -> +5V
- CON2 pad 7: VDD -> /SCL
- CON2 pad 8: /PCLK -> /SDA
- CON2 pad 9: /HSYNC -> /IRQ
- L1 pad 1: Net-(C8-Pad1) -> Net-(C3-Pad1)
- P1 pad 1: +12V -> VDD
- P1 pad 3: Net-(P1-Pad3) -> GND
- P1 pad 6: GND -> Net-(P1-Pad6)
- P1 pad 7: Net-(P1-Pad7) -> (no net)
- R1 pad 1: Net-(R1-Pad1) -> Net-(CON1-Pad13)
- R1 pad 2: Net-(C2-Pad1) -> GND
- R2 pad 1: Net-(R2-Pad1) -> Net-(P1-Pad5)
- R2 pad 2: Net-(C3-Pad1) -> VDD
- R3 pad 1: Net-(R3-Pad1) -> VDD
- R3 pad 2: Net-(C4-Pad1) -> Net-(BT1-Pad1)
- R4 pad 2: Net-(C5-Pad1) -> Net-(C6-Pad1)
- R5 pad 1: Net-(R5-Pad1) -> Net-(Q1-Pad1)
- R5 pad 2: +5V -> Net-(CON1-Pad36)
- R6 pad 1: Net-(CON2-Pad13) -> VDD
- R6 pad 2: GND -> Net-(Q1-Pad3)
- U1 pad 1: VDD -> Net-(L2-Pad1)
- U1 pad 10: /D5 -> Net-(L3-Pad1)
- U1 pad 11: /D6 -> VDD
- U1 pad 12: GND -> VDD
- U1 pad 13: /D7 -> GND
- U1 pad 14: VDD -> (no net)
- U1 pad 15: /NBL0 -> (no net)
- U1 pad 16: /WE# -> (no net)
- U1 pad 17: /CAS# -> (no net)
- U1 pad 18: /RAS# -> (no net)
- U1 pad 19: /CS# -> (no net)
- U1 pad 2: /D0 -> GND
- U1 pad 20: /BA0 -> (no net)
- U1 pad 21: /BA1 -> (no net)
- U1 pad 22: /A10 -> (no net)
- U1 pad 23: /A0 -> (no net)
- U1 pad 24: /A1 -> (no net)
- U1 pad 25: /A2 -> (no net)
- U1 pad 26: /A3 -> (no net)
- U1 pad 27: VDD -> (no net)
- U1 pad 28: GND -> (no net)
- U1 pad 29: /A4 -> (no net)
- U1 pad 3: VDD -> Net-(C1-Pad1)
- U1 pad 30: /A5 -> (no net)
- U1 pad 31: /A6 -> (no net)
- U1 pad 32: /A7 -> (no net)
- U1 pad 33: /A8 -> (no net)
- U1 pad 34: /A9 -> (no net)
- U1 pad 35: /A11 -> (no net)
- U1 pad 36: /A12 -> (no net)
- U1 pad 37: /CKE -> (no net)
- U1 pad 38: /CLK -> (no net)
- U1 pad 39: /NBL1 -> (no net)
- U1 pad 4: /D1 -> Net-(U1-Pad4)
- U1 pad 40: Net-(U1-Pad40) -> (no net)
- U1 pad 41: GND -> (no net)
- U1 pad 42: /D8 -> (no net)
- U1 pad 43: VDD -> (no net)
- U1 pad 44: /D9 -> (no net)
- U1 pad 45: /D10 -> (no net)
- U1 pad 46: GND -> (no net)
- U1 pad 47: /D11 -> (no net)
- U1 pad 48: /D12 -> (no net)
- U1 pad 49: VDD -> (no net)
- U1 pad 5: /D2 -> GND
- U1 pad 50: /D13 -> (no net)
- U1 pad 51: /D14 -> (no net)
- U1 pad 52: GND -> (no net)
- U1 pad 53: /D15 -> (no net)
- U1 pad 54: GND -> (no net)
- U1 pad 6: GND -> Net-(C2-Pad1)
- U1 pad 7: /D3 -> Net-(U1-Pad7)
- U1 pad 8: /D4 -> Net-(Q1-Pad3)
- U1 pad 9: VDD -> Net-(C9-Pad1)
- U2 pad 1: Net-(U2-Pad1) -> /SCK
- U2 pad 10: Net-(R2-Pad1) -> /A0
- U2 pad 100: Net-(U2-Pad100) -> /SCL
- U2 pad 101: Net-(U2-Pad101) -> /IRQ
- U2 pad 102: GND -> Net-(U2-Pad102)
- U2 pad 103: VDD -> /R2
- U2 pad 104: /D0 -> /R3
- U2 pad 105: /D1 -> Net-(P1-Pad4)
- U2 pad 106: /A12 -> Net-(C21-Pad2)
- U2 pad 107: Net-(U2-Pad107) -> GND
- U2 pad 108: /BA0 -> VDD
- U2 pad 109: /BA1 -> Net-(P1-Pad2)
- U2 pad 11: Net-(U2-Pad11) -> /A1
- U2 pad 110: /R5 -> Net-(U2-Pad110)
- U2 pad 111: /PCLK -> /R0
- U2 pad 112: /CLK -> Net-(U2-Pad112)
- U2 pad 113: GND -> Net-(U2-Pad113)
- U2 pad 114: VDD -> /D2
- U2 pad 115: /HSYNC -> /D3
- U2 pad 116: /G4 -> Net-(U2-Pad116)
- U2 pad 117: Net-(U2-Pad117) -> /G5
- U2 pad 12: Net-(U2-Pad12) -> /A2
- U2 pad 120: Net-(U2-Pad120) -> GND
- U2 pad 121: Net-(U2-Pad121) -> VDD
- U2 pad 122: /R2 -> /B0
- U2 pad 123: /R3 -> Net-(U2-Pad123)
- U2 pad 125: Net-(C1-Pad2) -> /G1
- U2 pad 126: GND -> /B1
- U2 pad 127: VDD -> /B2
- U2 pad 13: Net-(U2-Pad13) -> /A3
- U2 pad 130: Net-(U2-Pad130) -> GND
- U2 pad 131: /NSS -> VDD
- U2 pad 132: /SCK -> /CAS#
- U2 pad 133: /MISO -> Net-(U2-Pad133)
- U2 pad 134: /MOSI -> Net-(U2-Pad134)
- U2 pad 135: GND -> /CKE
- U2 pad 136: VDD -> /CS#
- U2 pad 138: Net-(U2-Pad138) -> GND
- U2 pad 139: /R0 -> /B4
- U2 pad 14: GND -> /A4
- U2 pad 140: Net-(U2-Pad140) -> /B5
- U2 pad 141: Net-(U2-Pad141) -> /NBL0
- U2 pad 142: /D2 -> /NBL1
- U2 pad 143: /D3 -> VDD
- U2 pad 144: Net-(U2-Pad144) -> VDD
- U2 pad 145: /G5 -> (no net)
- U2 pad 146: Net-(U2-Pad146) -> (no net)
- U2 pad 147: Net-(U2-Pad147) -> (no net)
- U2 pad 148: GND -> (no net)
- U2 pad 149: VDD -> (no net)
- U2 pad 15: VDD -> /A5
- U2 pad 150: /B0 -> (no net)
- U2 pad 151: Net-(U2-Pad151) -> (no net)
- U2 pad 152: Net-(U2-Pad152) -> (no net)
- U2 pad 153: /G1 -> (no net)
- U2 pad 154: /B1 -> (no net)
- U2 pad 155: /B2 -> (no net)
- U2 pad 156: Net-(U2-Pad156) -> (no net)
- U2 pad 157: Net-(U2-Pad157) -> (no net)
- U2 pad 158: GND -> (no net)
- U2 pad 159: VDD -> (no net)
- U2 pad 16: /A0 -> GND
- U2 pad 160: /CAS# -> (no net)
- U2 pad 161: Net-(U2-Pad161) -> (no net)
- U2 pad 162: Net-(U2-Pad162) -> (no net)
- U2 pad 163: /CKE -> (no net)
- U2 pad 164: /CS# -> (no net)
- U2 pad 165: Net-(U2-Pad165) -> (no net)
- U2 pad 166: Net-(U2-Pad166) -> (no net)
- U2 pad 167: /B4 -> (no net)
- U2 pad 168: /B5 -> (no net)
- U2 pad 169: /NBL0 -> (no net)
- U2 pad 17: /A1 -> VDD
- U2 pad 170: /NBL1 -> (no net)
- U2 pad 171: VDD -> (no net)
- U2 pad 172: VDD -> (no net)
- U2 pad 173: Net-(U2-Pad173) -> (no net)
- U2 pad 174: Net-(U2-Pad174) -> (no net)
- U2 pad 175: Net-(U2-Pad175) -> (no net)
- U2 pad 176: Net-(U2-Pad176) -> (no net)
- U2 pad 18: /A2 -> Net-(U2-Pad18)
- U2 pad 19: /A3 -> Net-(U2-Pad19)
- U2 pad 20: /A4 -> /SCL
- U2 pad 21: /A5 -> /SDI
- U2 pad 22: GND -> /EN
- U2 pad 23: VDD -> Net-(C5-Pad1)
- U2 pad 24: Net-(U2-Pad24) -> Net-(R4-Pad1)
- U2 pad 25: /SCL -> Net-(P1-Pad5)
- U2 pad 26: Net-(U2-Pad26) -> /WE#
- U2 pad 27: /SDI -> Net-(U2-Pad27)
- U2 pad 28: /EN -> Net-(U2-Pad28)
- U2 pad 29: Net-(R3-Pad1) -> Net-(U2-Pad29)
- U2 pad 3: Net-(U2-Pad3) -> /NSS
- U2 pad 30: Net-(R4-Pad1) -> VDD
- U2 pad 31: Net-(U2-Pad31) -> GND
- U2 pad 32: /WE# -> Net-(U2-Pad32)
- U2 pad 33: Net-(U2-Pad33) -> Net-(C3-Pad1)
- U2 pad 36: VDD -> Net-(U2-Pad36)
- U2 pad 37: GND -> /B3
- U2 pad 38: Net-(C6-Pad2) -> GND
- U2 pad 39: Net-(C8-Pad1) -> VDD
- U2 pad 4: Net-(U2-Pad4) -> /MISO
- U2 pad 40: Net-(U2-Pad40) -> /VSYNC
- U2 pad 42: Net-(U2-Pad42) -> /G0
- U2 pad 45: /SCL -> /CSB
- U2 pad 46: /SDA -> /R1
- U2 pad 47: /B3 -> /R4
- U2 pad 48: Net-(U2-Pad48) -> /RESETB
- U2 pad 49: VDD -> /RAS#
- U2 pad 5: Net-(U2-Pad5) -> /MOSI
- U2 pad 50: /VSYNC -> /A6
- U2 pad 51: Net-(U2-Pad51) -> GND
- U2 pad 52: /G0 -> VDD
- U2 pad 53: Net-(U2-Pad53) -> /A7
- U2 pad 54: Net-(U2-Pad54) -> /A8
- U2 pad 55: /CSB -> /A9
- U2 pad 56: /R1 -> /A10
- U2 pad 57: /R4 -> /A11
- U2 pad 58: /RESETB -> /D4
- U2 pad 59: /RAS# -> /D5
- U2 pad 6: Net-(U2-Pad6) -> Net-(BT1-Pad1)
- U2 pad 60: /A6 -> /D6
- U2 pad 63: /A7 -> /D7
- U2 pad 64: /A8 -> /D8
- U2 pad 65: /A9 -> /D9
- U2 pad 66: /A10 -> /D10
- U2 pad 67: /A11 -> /D11
- U2 pad 68: /D4 -> /D12
- U2 pad 69: /D5 -> /G2
- U2 pad 70: /D6 -> /G3
- U2 pad 71: GND -> Net-(C19-Pad2)
- U2 pad 73: /D7 -> Net-(U2-Pad73)
- U2 pad 74: /D8 -> Net-(U2-Pad74)
- U2 pad 75: /D9 -> Net-(U2-Pad75)
- U2 pad 76: /D10 -> Net-(U2-Pad76)
- U2 pad 77: /D11 -> /D13
- U2 pad 78: /D12 -> /D14
- U2 pad 79: /G2 -> /D15
- U2 pad 8: Net-(U2-Pad8) -> Net-(C7-Pad1)
- U2 pad 80: /G3 -> Net-(U2-Pad80)
- U2 pad 81: Net-(C10-Pad1) -> Net-(U2-Pad81)
- U2 pad 82: VDD -> Net-(U2-Pad82)
- U2 pad 83: /IRQ -> GND
- U2 pad 84: /SCL -> VDD
- U2 pad 85: /SDA -> /D0
- U2 pad 86: Net-(U2-Pad86) -> /D1
- U2 pad 87: Net-(U2-Pad87) -> /A12
- U2 pad 89: Net-(U2-Pad89) -> /BA0
- U2 pad 9: Net-(R1-Pad1) -> Net-(C8-Pad1)
- U2 pad 90: GND -> /BA1
- U2 pad 91: VDD -> /R5
- U2 pad 92: Net-(U2-Pad92) -> /PCLK
- U2 pad 93: Net-(U2-Pad93) -> /CLK
- U2 pad 94: Net-(U2-Pad94) -> GND
- U2 pad 95: Net-(U2-Pad95) -> VDD
- U2 pad 96: /D13 -> /HSYNC
- U2 pad 97: /D14 -> /G4
- U2 pad 98: /D15 -> Net-(U2-Pad98)
- U2 pad 99: Net-(U2-Pad99) -> /SDA
- U3 pad 1: /NSS -> Net-(U2-Pad74)
- U3 pad 2: /MISO -> GND
- U3 pad 3: VDD -> +5V
- U3 pad 4: GND -> Net-(U2-Pad73)
- U3 pad 6: /SCK -> Net-(P2-Pad7)
- U3 pad 7: VDD -> Net-(P2-Pad2)
- U3 pad 8: VDD -> GND
- U4 pad 1: Net-(U2-Pad93) -> GND
- U4 pad 2: GND -> +5V
- U4 pad 3: +5V -> +12V
- U4 pad 4: Net-(U2-Pad92) -> (no net)
- U4 pad 5: Net-(U4-Pad5) -> (no net)
- U4 pad 6: Net-(P1-Pad7) -> (no net)
- U4 pad 7: Net-(P1-Pad2) -> (no net)
- U4 pad 8: GND -> (no net)
- U5 pad 1: /SCL -> Net-(U5-Pad1)
- U5 pad 10: Net-(M2-Pad1) -> Net-(U5-Pad10)
- U5 pad 11: Net-(M2-Pad2) -> Net-(U5-Pad11)
- U5 pad 12: Net-(M2-Pad3) -> GND
- U5 pad 13: Net-(M2-Pad4) -> Net-(M2-Pad1)
- U5 pad 14: Net-(M1-Pad1) -> Net-(M2-Pad2)
- U5 pad 15: Net-(M1-Pad2) -> Net-(M2-Pad3)
- U5 pad 16: Net-(M1-Pad3) -> Net-(M2-Pad4)
- U5 pad 17: Net-(M1-Pad4) -> Net-(U5-Pad17)
- U5 pad 18: +5V -> Net-(U5-Pad18)
- U5 pad 2: /SDA -> GND
- U5 pad 4: GND -> Net-(M1-Pad1)
- U5 pad 5: GND -> Net-(M1-Pad2)
- U5 pad 6: Net-(R5-Pad1) -> Net-(M1-Pad3)
- U5 pad 7: Net-(U5-Pad7) -> Net-(M1-Pad4)
- U5 pad 9: GND -> Net-(U5-Pad9)
- U6 pad 1: Net-(L2-Pad1) -> GND
- U6 pad 10: Net-(L3-Pad1) -> (no net)
- U6 pad 11: VDD -> (no net)
- U6 pad 12: VDD -> (no net)
- U6 pad 13: GND -> (no net)
- U6 pad 2: GND -> VDD
- U6 pad 3: Net-(C11-Pad1) -> +12V
- U6 pad 4: Net-(U6-Pad4) -> (no net)
- U6 pad 5: GND -> (no net)
- U6 pad 6: Net-(C13-Pad1) -> (no net)
- U6 pad 7: Net-(U6-Pad7) -> (no net)
- U6 pad 8: Net-(Q1-Pad3) -> (no net)
- U6 pad 9: Net-(C12-Pad1) -> (no net)
- U7 pad 1: GND -> VDD
- U7 pad 2: +5V -> /D0
- U7 pad 3: +12V -> VDD
- U7 pad 4: (no net) -> /D1
- U8 pad 1: GND -> /NSS
- U8 pad 2: VDD -> /MISO
- U8 pad 3: +12V -> VDD
- U8 pad 4: (no net) -> GND
- Y1 pad 1: Net-(C2-Pad1) -> Net-(C5-Pad1)
- Y1 pad 2: Net-(C3-Pad1) -> Net-(C6-Pad1)
- Y2 pad 1: Net-(C4-Pad1) -> Net-(C7-Pad1)
- Y2 pad 2: Net-(C5-Pad1) -> Net-(C8-Pad1)

Commit message: regeneraed netlist
Parts:
- added C34: C, Capacitors_SMD:C_0603, F.Cu at (75.0, 70.1)
- C13: value C -> 10uF
- C14, C15, C16, C17: footprint Capacitors_SMD:c_elec_4x5.3 -> Capacitors_SMD:C_0603
- C19, C21: value 2.2uF -> C
- C20, C22: value C -> 2.2uF
- C24, C29: value 10uF -> C; footprint Capacitors_SMD:c_elec_4x5.3 -> Capacitors_SMD:C_0603
- C25, C32: value C -> 10uF; footprint Capacitors_SMD:C_0603 -> Capacitors_SMD:c_elec_4x5.3
- C3: footprint Capacitors_SMD:C_0603 -> Capacitors_SMD:c_elec_4x5.8
- C6: footprint Capacitors_Tantalum_SMD:TantalC_SizeB_EIA-3528_Wave -> Capacitors_SMD:C_0603
- C8: footprint Capacitors_Tantalum_SMD:TantalC_SizeA_EIA-3216_Wave -> Capacitors_SMD:C_0603
- C9: value 2x10uF -> 10uF
- CON1: footprint uberdashboard:BM10NB(0.8)-10DS-0.4V(51) -> uberdashboard:BM10NB(0.8)-40DS-0.4V(51)
- CON2: footprint uberdashboard:BM10NB(0.8)-40DS-0.4V(51) -> uberdashboard:BM10NB(0.8)-10DS-0.4V(51)
- P1: footprint Pin_Headers:Pin_Header_Straight_1x07 -> Pin_Headers:Pin_Header_Straight_1x06
- R1, R2, R3, R4, R5, R6: footprint Resistors_SMD:R_0805 -> Resistors_SMD:R_0603
- U1: footprint uberdashboard:TSOP54 -> Housings_DFN_QFN:QFN-12-1EP_3x3mm_Pitch0.5mm
- U2: footprint Housings_QFP:LQFP-176_24x24mm_Pitch0.5mm -> Housings_QFP:LQFP-144_20x20mm_Pitch0.5mm
- U3: footprint Housings_SOIC:SOIC-8_3.9x4.9mm_Pitch1.27mm -> Power_Integrations:SO-8
- U4: footprint Power_Integrations:SO-8 -> TO_SOT_Packages_SMD:SOT-223
- U5: footprint Housings_SOIC:SOIC-18_7.5x11.6mm_Pitch1.27mm -> Housings_SOIC:SOIC-24_7.5x15.4mm_Pitch1.27mm
- U6: footprint Housings_DFN_QFN:QFN-12-1EP_3x3mm_Pitch0.5mm -> TO_SOT_Packages_SMD:SOT-223
- U7: footprint TO_SOT_Packages_SMD:SOT-223 -> uberdashboard:TSOP54
- U8: footprint TO_SOT_Packages_SMD:SOT-223 -> Housings_SOIC:SOIC-8_3.9x4.9mm_Pitch1.27mm
- Y1: footprint Crystals:Crystal_Watch -> Crystals:Crystal_HC49-SD_SMD
- Y2: footprint Crystals:Crystal_HC49-SD_SMD -> Crystals:Crystal_Round_Horizontal_2mm
- moved C32 42.4 mm to (34.8, 56.5)
- moved U5 40.1 mm to (78.9, 7.00), turned to 90 degrees
- moved U1 36.5 mm to (56.3, 44.8)
- moved Y1 18.1 mm to (24.2, 25.7)
- moved C7 14.5 mm to (32.1, 31.0)
- moved U7 14.3 mm to (95.8, 40.3), turned to 90 degrees
- moved C28 12.2 mm to (70.0, 59.0)
- moved C3 11.0 mm to (23.1, 17.6)
- moved C8 9.12 mm to (32.0, 29.1), turned to 0 degrees
- moved C31 2.84 mm to (34.8, 50.8)
Connections:
- C13 pad 1: VDD -> Net-(C13-Pad1)
- C16 pad 1: GND -> VDD
- C16 pad 2: VDD -> GND
- C19 pad 2: Net-(C19-Pad2) -> VDD
- C20 pad 2: VDD -> Net-(C20-Pad2)
- C21 pad 2: Net-(C21-Pad2) -> VDD
- C22 pad 2: VDD -> Net-(C22-Pad2)
- C24 pad 1: +12V -> GND
- C24 pad 2: GND -> VDD
- C25 pad 1: VDD -> +12V
- C29 pad 1: +5V -> VDD
- C30 pad 1: +12V -> +5V
- C31 pad 1: VDD -> +12V
- C32 pad 1: GND -> VDD
- C32 pad 2: VDD -> GND
- C9 pad 1: Net-(C9-Pad1) -> Net-(C13-Pad1)
- CON1 pad 2: Net-(C9-Pad1) -> Net-(C13-Pad1)
- CON1 pad 4: Net-(C9-Pad1) -> Net-(C13-Pad1)
- U1 pad 9: Net-(C9-Pad1) -> Net-(C13-Pad1)
- U2 pad 106: Net-(C21-Pad2) -> Net-(C22-Pad2)
- U2 pad 71: Net-(C19-Pad2) -> Net-(C20-Pad2)

Commit message: Added files via upload
Parts:
- M1, M2: moved to B.Cu
- R8: moved to F.Cu
- moved C33 39.1 mm to (84.0, 32.0)
- moved R5 38.9 mm to (81.0, 44.0), turned to 270 degrees
- moved P2 34.0 mm to (77.0, 3.00)
- moved C1 24.2 mm to (59.0, 43.0), turned to 180 degrees
- moved BT1 23.0 mm to (101.0, 57.0), turned to 90 degrees
- moved C24 22.1 mm to (94.0, 32.0)
- moved C25 19.6 mm to (88.0, 45.0)
- moved C20 19.2 mm to (70.0, 44.0), turned to 180 degrees
- moved R8 18.6 mm to (76.0, 43.0), turned to 180 degrees
- moved U3 18.4 mm to (79.0, 36.0), turned to 270 degrees
- moved C15 18.4 mm to (114.0, 31.0), turned to 270 degrees
- moved C34 17.5 mm to (82.0, 54.0), turned to 180 degrees
- moved C22 16.5 mm to (73.0, 53.0), turned to 90 degrees
- moved C16 16.3 mm to (121.0, 50.0), turned to 180 degrees
- moved C29 16.3 mm to (82.0, 57.0)
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Other:
- board size 150 x 60 mm -> 255 x 126 mm

Commit message: i2c to vdd
Parts:
- added R5: 1K, Resistors_SMD:R_0603, F.Cu at (76.0, 43.0)
- added R6: 10K, Resistors_SMD:R_0603, B.Cu at (66.0, 29.0)
- R7: value 10K -> 4.7k; footprint Resistors_SMD:R_0805 -> Resistors_SMD:R_0603; moved to F.Cu
- R8: value 1K -> 4.7k; footprint Resistors_SMD:R_0805 -> Resistors_SMD:R_0603
- moved R8 26.8 mm to (73.2, 16.3), turned to 0 degrees
- moved R7 16.1 mm to (70.6, 13.6), turned to 0 degrees
- moved U5 2.06 mm to (85.6, 17.3)
Connections:
- CON2 pad 2: Net-(CON2-Pad2) -> (no net)
- CON2 pad 4: Net-(CON2-Pad4) -> (no net)
- P1 pad 6: Net-(P1-Pad6) -> (no net)
- P2 pad 3: Net-(P2-Pad3) -> (no net)
- P2 pad 4: Net-(P2-Pad4) -> (no net)
- P2 pad 5: Net-(P2-Pad5) -> (no net)
- R7 pad 2: Net-(Q1-Pad3) -> /SDA
- R8 pad 1: Net-(Q1-Pad1) -> VDD
- R8 pad 2: Net-(CON2-Pad36) -> /SCL
- U1 pad 4: Net-(U1-Pad4) -> (no net)
- U1 pad 7: Net-(U1-Pad7) -> (no net)
- U2 pad 102: Net-(U2-Pad102) -> (no net)
- U2 pad 110: Net-(U2-Pad110) -> (no net)
- U2 pad 112: Net-(U2-Pad112) -> (no net)
- U2 pad 113: Net-(U2-Pad113) -> (no net)
- U2 pad 116: Net-(U2-Pad116) -> (no net)
- U2 pad 118: Net-(U2-Pad118) -> (no net)
- U2 pad 119: Net-(U2-Pad119) -> (no net)
- U2 pad 123: Net-(U2-Pad123) -> (no net)
- U2 pad 124: Net-(U2-Pad124) -> (no net)
- U2 pad 128: Net-(U2-Pad128) -> (no net)
- U2 pad 129: Net-(U2-Pad129) -> (no net)
- U2 pad 133: Net-(U2-Pad133) -> (no net)
- U2 pad 134: Net-(U2-Pad134) -> (no net)
- U2 pad 137: Net-(U2-Pad137) -> (no net)
- U2 pad 18: Net-(U2-Pad18) -> (no net)
- U2 pad 19: Net-(U2-Pad19) -> (no net)
- U2 pad 2: Net-(U2-Pad2) -> (no net)
- U2 pad 27: Net-(U2-Pad27) -> (no net)
- U2 pad 28: Net-(U2-Pad28) -> (no net)
- U2 pad 29: Net-(U2-Pad29) -> (no net)
- U2 pad 32: Net-(U2-Pad32) -> (no net)
- U2 pad 34: Net-(U2-Pad34) -> (no net)
- U2 pad 35: Net-(U2-Pad35) -> (no net)
- U2 pad 36: Net-(U2-Pad36) -> (no net)
- U2 pad 41: Net-(U2-Pad41) -> (no net)
- U2 pad 43: Net-(U2-Pad43) -> (no net)
- U2 pad 44: Net-(U2-Pad44) -> (no net)
- U2 pad 7: Net-(U2-Pad7) -> (no net)
- U2 pad 75: Net-(U2-Pad75) -> (no net)
- U2 pad 76: Net-(U2-Pad76) -> (no net)
- U2 pad 80: Net-(U2-Pad80) -> (no net)
- U2 pad 81: Net-(U2-Pad81) -> (no net)
- U2 pad 82: Net-(U2-Pad82) -> (no net)
- U2 pad 88: Net-(U2-Pad88) -> (no net)
- U2 pad 98: Net-(U2-Pad98) -> (no net)
- U3 pad 5: Net-(U3-Pad5) -> (no net)
- U5 pad 1: Net-(U5-Pad1) -> (no net)
- U5 pad 10: Net-(U5-Pad10) -> (no net)
- U5 pad 11: Net-(U5-Pad11) -> (no net)
- U5 pad 17: Net-(U5-Pad17) -> (no net)
- U5 pad 18: Net-(U5-Pad18) -> (no net)
- U5 pad 19: Net-(U5-Pad19) -> (no net)
- U5 pad 20: Net-(U5-Pad20) -> (no net)
- U5 pad 8: Net-(U5-Pad8) -> (no net)
- U5 pad 9: Net-(U5-Pad9) -> (no net)
- U7 pad 40: Net-(U7-Pad40) -> (no net)
Other:
- board size 255 x 126 mm -> 150 x 60 mm

Commit message: C19
Parts:
- added C19: 0.1uF, Capacitors_SMD:C_0603, F.Cu at (75.0, 70.1)
- C11, C12, C14, C15, C16, C17, C18: value C -> 0.1uF
- C20: renamed from C19; value C -> 0.1uF
- C22: renamed from C21; value C -> 0.1uF
- C27: renamed from C26; value C -> 0.1uF
- C28: renamed from C27; value C -> 0.1uF
- C29: renamed from C28; value C -> 0.1uF
- C30: renamed from C29; value C -> 0.1uF
- C34: renamed from C33; value C -> 0.1uF
- C35: renamed from C34; value C -> 0.1uF
- renumbered C20 to C21, C22 to C23, C23 to C24, C24 to C25, C25 to C26, C30 to C31, C31 to C32, C32 to C33

Commit message: reannotation and removed unncessary R
Parts:
- removed the R5 at (76.0, 43.0)
- removed the R6 at (58.0, 28.0)
- moved C19 19.6 mm to (60.8, 56.5)
- moved U6 11.2 mm to (64.2, 13.1)
- moved R6 9.63 mm to (56.4, 28.2), turned to 0 degrees
- moved C13 5.80 mm to (57.5, 13.4)
- moved L2 1.63 mm to (52.2, 27.1)
- moved CON2 1.32 mm to (61.3, 33.2)
- moved Q1 1.20 mm to (62.2, 28.0)
Changed lines of the file:
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@@
 (kicad_pcb (version 4) (host pcbnew 4.0.2-4+6225~38~ubuntu15.10.1-stable)
   (general
-    (links 274)
-    (no_connects 274)
+    (links 270)
+    (no_connects 270)
     (area -0.075001 -0.075001 150.075001 60.075001)
     (thickness 1.6)
@@
     (tracks 0)
     (zones 0)
-    (modules 66)
+    (modules 64)
     (nets 109)
   )
@@
   )
   (module Capacitors_SMD:C_0603 (layer B.Cu)
-    (at 59 19 180)
+    (at 57.5 13.4 180)
     (descr "Capacitor SMD 0603, reflow soldering, AVX (see smccp.pdf)")
     (tags "capacitor 0603")
@@
   )
   (module Resistors_SMD:R_1812 (layer B.Cu)
-    (at 51 26 270)
+    (at 52.2 27.1 270)
     (descr "Resistor SMD 1812, flow soldering, Panasonic (see ERJ12)")
     (tags "resistor 1812")
@@
   )
   (module TO_SOT_Packages_SMD:SOT-23 (layer B.Cu)
-    (at 61 28 90)
+    (at 62.2 28 90)
     (descr "SOT-23, Standard")
     (tags SOT-23)
@@
   )
   (module "uberdashboard:BM10NB(0.8)-10DS-0.4V(51)" (layer B.Cu)
-    (at 60 33)
+    (at 61.3 33.2)
     (fp_text reference CON2 (at 0 -2.7) (layer B.SilkS)
       (effects (font (size 1 1) (thickness 0.15)) (justify mirror))
@@
   )
   (module TO_SOT_Packages_SMD:SOT-223 (layer B.Cu)
-    (at 59 23)
+    (at 64.2 13.1)
     (descr "module CMS SOT223 4 pins")
     (tags "CMS SOT")
@@
   )
   (module Resistors_SMD:R_0603 (layer B.Cu)
-    (at 58 28 90)
+    (at 56.4 28.2)
     (descr "Resistor SMD 0603, reflow soldering, Vishay (see dcrcw.pdf)")
     (tags "resistor 0603")
     (attr smd)
-    (fp_text reference R6 (at 0 1.9 90) (layer B.SilkS)
-      (effects (font (size 1 1) (thickness 0.15)) (justify mirror))
-    )
-    (fp_text value 10K (at 0 -1.9 90) (layer B.Fab)
+    (fp_text reference R6 (at 0 1.9) (layer B.SilkS)
+      (effects (font (size 1 1) (thickness 0.15)) (justify mirror))
+    )
+    (fp_text value 10K (at 0 -1.9) (layer B.Fab)
       (effects (font (size 1 1) (thickness 0.15)) (justify mirror))
     )
@@
     (fp_line (start 0.5 -0.675) (end -0.5 -0.675) (layer B.SilkS) (width 0.15))
     (fp_line (start -0.5 0.675) (end 0.5 0.675) (layer B.SilkS) (width 0.15))
-    (pad 1 smd rect (at -0.75 0 90) (size 0.5 0.9) (layers B.Cu B.Paste B.Mask)
-      (net 8 VDD))
-    (pad 2 smd rect (at 0.75 0 90) (size 0.5 0.9) (layers B.Cu B.Paste B.Mask)
-      (net 37 "Net-(Q1-Pad3)"))
-    (model Resistors_SMD.3dshapes/R_0603.wrl
-      (at (xyz 0 0 0))
-      (scale (xyz 1 1 1))
-      (rotate (xyz 0 0 0))
-    )
-  )
-  (module Resistors_SMD:R_0603 (layer F.Cu)
-    (at 76 43 180)
-    (descr "Resistor SMD 0603, reflow soldering, Vishay (see dcrcw.pdf)")
-    (tags "resistor 0603")
-    (attr smd)
-    (fp_text reference R5 (at 0 -1.9 180) (layer F.SilkS)
-      (effects (font (size 1 1) (thickness 0.15)))
-    )
-    (fp_text value 1K (at 0 1.9 180) (layer F.Fab)
-      (effects (font (size 1 1) (thickness 0.15)))
-    )
-    (fp_line (start -1.3 -0.8) (end 1.3 -0.8) (layer F.CrtYd) (width 0.05))
-    (fp_line (start -1.3 0.8) (end 1.3 0.8) (layer F.CrtYd) (width 0.05))
-    (fp_line (start -1.3 -0.8) (end -1.3 0.8) (layer F.CrtYd) (width 0.05))
-    (fp_line (start 1.3 -0.8) (end 1.3 0.8) (layer F.CrtYd) (width 0.05))
-    (fp_line (start 0.5 0.675) (end -0.5 0.675) (layer F.SilkS) (width 0.15))
-    (fp_line (start -0.5 -0.675) (end 0.5 -0.675) (layer F.SilkS) (width 0.15))
-    (pad 1 smd rect (at -0.75 0 180) (size 0.5 0.9) (layers F.Cu F.Paste F.Mask)
-      (net 36 "Net-(Q1-Pad1)"))
-    (pad 2 smd rect (at 0.75 0 180) (size 0.5 0.9) (layers F.Cu F.Paste F.Mask)
-      (net 69 "Net-(CON1-Pad36)"))
-    (model Resistors_SMD.3dshapes/R_0603.wrl
-      (at (xyz 0 0 0))
-      (scale (xyz 1 1 1))
-      (rotate (xyz 0 0 0))
-    )
-  )
-  (module Resistors_SMD:R_0603 (layer B.Cu)
-    (at 66 29 180)
-    (descr "Resistor SMD 0603, reflow soldering, Vishay (see dcrcw.pdf)")
-    (tags "resistor 0603")
-    (attr smd)
-    (fp_text reference R6 (at 0 1.9 180) (layer B.SilkS)
-      (effects (font (size 1 1) (thickness 0.15)) (justify mirror))
-    )
-    (fp_text value 10K (at 0 -1.9 180) (layer B.Fab)
-      (effects (font (size 1 1) (thickness 0.15)) (justify mirror))
-    )
-    (fp_line (start -1.3 0.8) (end 1.3 0.8) (layer B.CrtYd) (width 0.05))
-    (fp_line (start -1.3 -0.8) (end 1.3 -0.8) (layer B.CrtYd) (width 0.05))
-    (fp_line (start -1.3 0.8) (end -1.3 -0.8) (layer B.CrtYd) (width 0.05))
-    (fp_line (start 1.3 0.8) (end 1.3 -0.8) (layer B.CrtYd) (width 0.05))
-    (fp_line (start 0.5 -0.675) (end -0.5 -0.675) (layer B.SilkS) (width 0.15))
-    (fp_line (start -0.5 0.675) (end 0.5 0.675) (layer B.SilkS) (width 0.15))
-    (pad 1 smd rect (at -0.75 0 180) (size 0.5 0.9) (layers B.Cu B.Paste B.Mask)
-      (net 8 VDD))
-    (pad 2 smd rect (at 0.75 0 180) (size 0.5 0.9) (layers B.Cu B.Paste B.Mask)
+    (pad 1 smd rect (at -0.75 0) (size 0.5 0.9) (layers B.Cu B.Paste B.Mask)
+      (net 8 VDD))
+    (pad 2 smd rect (at 0.75 0) (size 0.5 0.9) (layers B.Cu B.Paste B.Mask)
       (net 37 "Net-(Q1-Pad3)"))
     (model Resistors_SMD.3dshapes/R_0603.wrl
@@
   )
   (module Capacitors_SMD:C_0603 (layer F.Cu)
-    (at 75 70.075001)
-    (descr "Capacitor SMD 0603, reflow soldering, AVX (see smccp.pdf)")
-    (tags "capacitor 0603")
+    (at 60.8 56.5)
+    (descr "Capacitor SMD 0603, reflow soldering, AVX (see smccp.pdf)")
+    (tags "capacitor 0603")

Commit message: Added files via upload
Parts:
- C1, C9, CON1, R1, R5, R7, R8, U1, U5: moved to B.Cu
- C12, C4, C6, R3, U6: moved to F.Cu
- moved C31 67.5 mm to (43.0, 42.0), turned to 270 degrees
- moved C14 66.2 mm to (55.0, 16.0), turned to 90 degrees
- moved BT1 63.5 mm to (48.0, 22.0), turned to 270 degrees
- moved P1 63.3 mm to (89.0, 3.00)
- moved C15 58.5 mm to (57.0, 44.0)
- moved C16 58.3 mm to (63.0, 44.0), turned to 270 degrees
- moved U6 54.5 mm to (26.0, 52.0), turned to 90 degrees
- moved P2 54.3 mm to (71.0, 57.0)
- moved U4 53.1 mm to (45.0, 53.0), turned to 180 degrees
- moved C35 51.7 mm to (121.0, 20.0)
- moved C22 51.6 mm to (77.0, 19.0), turned to 180 degrees
- moved C30 42.5 mm to (101.0, 19.0)
- moved U8 38.6 mm to (89.0, 17.0), turned to 180 degrees
- moved C29 38.2 mm to (101.0, 30.0), turned to 0 degrees
- moved C34 37.3 mm to (121.0, 27.0), turned to 180 degrees
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