File: uberdashboard.kicad_pcb (KiCad board)
At the start: 2 copper layers, 150 x 60 mm, 64 parts, among them CON1 AMOLED-BM10NB(0.8)-40DS-0.4V(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, CON2 TOUCH-BM10NB(0.8)-10DS-0.4V(5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, M1 VID23-03, M2 VID23-03, P1 CONN_01X06, P2 CONN_ROUNDX07, Q1 BC817-40, U1 STOD13AS, U2 STM32F429ZIT6, U3 MCP2551-I/SN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

Commit message: misplaced
Parts:
- CON2: moved to F.Cu
- moved CON2 31.5 mm to (87.1, 47.2)
- moved CON1 4.42 mm to (55.5, 30.3), turned to 180 degrees

Commit message: Added files via upload
Parts:
- CON2: moved to B.Cu
- moved C33 77.1 mm to (45.5, -20.5), turned to 90 degrees
- moved C32 72.2 mm to (51.5, -20.5), turned to 90 degrees
- moved Y1 67.5 mm to (65.0, -22.0), turned to 0 degrees
- moved U4 64.6 mm to (48.5, -11.5), turned to 90 degrees
- moved C31 57.9 mm to (59.5, -13.5), turned to 180 degrees
- moved C26 57.8 mm to (47.5, -3.50), turned to 180 degrees
- moved C5 56.6 mm to (66.5, -15.5), turned to 90 degrees
- moved C6 55.1 mm to (70.5, -15.5), turned to 90 degrees
- moved Y2 54.0 mm to (75.5, -15.5), turned to 0 degrees
- moved C12 51.7 mm to (65.5, -11.5), turned to 180 degrees
- moved U6 51.0 mm to (48.0, 6.00), turned to 180 degrees
- moved C3 50.8 mm to (56.5, -5.50), turned to 90 degrees
- moved C4 50.3 mm to (61.5, -8.50), turned to 90 degrees
- moved P2 50.1 mm to (44.5, 14.5), turned to 0 degrees
- moved R4 49.9 mm to (69.5, -11.5), turned to 0 degrees
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Other:
- board size 150 x 60 mm -> 150 x 95 mm

Commit message: Touch connector
Parts:
- CON2: moved to F.Cu
- moved CON2 14.2 mm to (89.0, 20.0), turned to 180 degrees
Changed lines of the file:
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@@
-(kicad_pcb (version 4) (host pcbnew 4.0.1-stable)
+(kicad_pcb (version 4) (host pcbnew 4.0.2-4+6225~38~ubuntu15.10.1-stable)
   (general
     (links 270)
     (no_connects 270)
-    (area -0.075001 -2.108334 150.075001 63.727381)
+    (area -0.075001 -35.075001 150.075001 60.075001)
     (thickness 1.6)
     (drawings 9)
@@
     (pad "" connect rect (at 4.55 1.45) (size 0.92 0.55) (layers B.Cu B.Mask))
   )
-  (module "uberdashboard:BM10NB(0.8)-10DS-0.4V(51)" (layer B.Cu)
-    (at 78.5 10.5 270)
-    (fp_text reference CON2 (at 0 -2.7 270) (layer B.SilkS)
-      (effects (font (size 1 1) (thickness 0.15)) (justify mirror))
-    )
-    (fp_text value "TOUCH-BM10NB(0.8)-10DS-0.4V(51)" (at 0 2.85 270) (layer B.Fab)
-      (effects (font (size 1 1) (thickness 0.15)) (justify mirror))
-    )
-    (pad "" connect rect (at -1.6 1.45 270) (size 0.92 0.55) (layers B.Cu B.Mask))
-    (pad "" connect rect (at -1.6 -1.45 270) (size 0.92 0.55) (layers B.Cu B.Mask))
-    (pad "" connect rect (at 1.6 -1.45 270) (size 0.92 0.55) (layers B.Cu B.Mask))
-    (pad 10 connect rect (at -0.8 1.4 270) (size 0.23 0.45) (layers B.Cu B.Mask)
-      (net 1 GND))
-    (pad 9 connect rect (at -0.4 1.4 270) (size 0.23 0.45) (layers B.Cu B.Mask)
+  (module "uberdashboard:BM10NB(0.8)-10DS-0.4V(51)" (layer F.Cu)
+    (at 89 20 180)
+    (fp_text reference CON2 (at 0 2.7 180) (layer F.SilkS)
+      (effects (font (size 1 1) (thickness 0.15)))
+    )
+    (fp_text value "TOUCH-BM10NB(0.8)-10DS-0.4V(51)" (at 0 -2.85 180) (layer F.Fab)
+      (effects (font (size 1 1) (thickness 0.15)))
+    )
+    (pad "" connect rect (at -1.6 -1.45 180) (size 0.92 0.55) (layers F.Cu F.Mask))
+    (pad "" connect rect (at -1.6 1.45 180) (size 0.92 0.55) (layers F.Cu F.Mask))
+    (pad "" connect rect (at 1.6 1.45 180) (size 0.92 0.55) (layers F.Cu F.Mask))
+    (pad 10 connect rect (at -0.8 -1.4 180) (size 0.23 0.45) (layers F.Cu F.Mask)
+      (net 1 GND))
+    (pad 9 connect rect (at -0.4 -1.4 180) (size 0.23 0.45) (layers F.Cu F.Mask)
       (net 9 /IRQ))
-    (pad 7 connect rect (at 0.4 1.4 270) (size 0.23 0.45) (layers B.Cu B.Mask)
+    (pad 7 connect rect (at 0.4 -1.4 180) (size 0.23 0.45) (layers F.Cu F.Mask)
       (net 10 /SCL))
-    (pad 8 connect rect (at 0 1.4 270) (size 0.23 0.45) (layers B.Cu B.Mask)
+    (pad 8 connect rect (at 0 -1.4 180) (size 0.23 0.45) (layers F.Cu F.Mask)
       (net 11 /SDA))
-    (pad 6 connect rect (at 0.8 1.4 270) (size 0.23 0.45) (layers B.Cu B.Mask)
-      (net 1 GND))
-    (pad 5 connect rect (at 0.8 -1.4 270) (size 0.23 0.45) (layers B.Cu B.Mask)
+    (pad 6 connect rect (at 0.8 -1.4 180) (size 0.23 0.45) (layers F.Cu F.Mask)
+      (net 1 GND))
+    (pad 5 connect rect (at 0.8 1.4 180) (size 0.23 0.45) (layers F.Cu F.Mask)
       (net 7 +5V))
-    (pad 3 connect rect (at 0 -1.4 270) (size 0.23 0.45) (layers B.Cu B.Mask)
+    (pad 3 connect rect (at 0 1.4 180) (size 0.23 0.45) (layers F.Cu F.Mask)
       (net 7 +5V))
-    (pad 4 connect rect (at 0.4 -1.4 270) (size 0.23 0.45) (layers B.Cu B.Mask))
-    (pad 2 connect rect (at -0.4 -1.4 270) (size 0.23 0.45) (layers B.Cu B.Mask))
-    (pad 1 connect rect (at -0.8 -1.4 270) (size 0.23 0.45) (layers B.Cu B.Mask)
-      (net 1 GND))
-    (pad "" connect rect (at 1.6 1.45 270) (size 0.92 0.55) (layers B.Cu B.Mask))
+    (pad 4 connect rect (at 0.4 1.4 180) (size 0.23 0.45) (layers F.Cu F.Mask))
+    (pad 2 connect rect (at -0.4 1.4 180) (size 0.23 0.45) (layers F.Cu F.Mask))
+    (pad 1 connect rect (at -0.8 1.4 180) (size 0.23 0.45) (layers F.Cu F.Mask)
+      (net 1 GND))
+    (pad "" connect rect (at 1.6 -1.45 180) (size 0.92 0.55) (layers F.Cu F.Mask))
   )
   (module Pin_Headers:Pin_Header_Straight_1x06 (layer F.Cu)
